File: hardware/kicad/08_connectors.kicad_sch (KiCad schematic)
At the start: 0 parts

Commit message: docs: organize hardware readiness for final KiCad handoff
Other:
- note added: "USB-C, microSD, display/touch and expansion connectors. C1 Rev J is reviewed; connector geometry and samples still gate footprints."
- note removed: "USB-C, microSD, display/touch and expansion connectors. Exact display C1 drawing remains required."
Changed lines of the file:
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@@
 	(paper "A4")
 	(title_block (title "08 Connectors") (rev "architecture-gate"))
-	(text "USB-C, microSD, display/touch and expansion connectors. Exact display C1 drawing remains required." (exclude_from_sim no) (at 25.4 30.48 0) (effects (font (size 1.27 1.27)) (justify left bottom)))
+	(text "USB-C, microSD, display/touch and expansion connectors. C1 Rev J is reviewed; connector geometry and samples still gate footprints." (exclude_from_sim no) (at 25.4 30.48 0) (effects (font (size 1.27 1.27)) (justify left bottom)))
 	(sheet_instances (path "/" (page "1")))
 	(embedded_fonts no)
