File: candidates/claude-oneshot-revA/kicad/05_display.kicad_sch (KiCad schematic)
At the start: 25 parts, among them J3 XF3M-4015-1B (TFT 40p FPC), J4 XF3M-0615-1B (CTP 6p FPC), U14 SN74AXC4T245PWR, U15 SN74LVC1G07DBVR, U16 TPS61169DCKR

Commit message: docs: show one-shot candidate renders and schematic in README, fix 3D models
Root README gains a status table for the Claude one-shot candidate, 3D and
enclosure renders, PCB copper view, all 12 schematic sheets as images and
step-by-step instructions (folders) to open the KiCad project or the STEP
files. Candidate README gets the same gallery and KiCad instructions.

3D: envelope STEP models for parts whose footprint had no model in the
KiCad 10.0.6 install (MAX-M10S, ICM-42688-P, MMC5983MA, BMP581, TPD1E0B04,
TPS259474L RPW, TUSB320LAI, Coilcraft inductors, SHT40), so the board STEP
and the Alt+3 view are complete. Routing unchanged; DRC 1 reviewed error,
11 unconnected, parity 0.

Co-Authored-By: Claude Opus 5.5 <noreply@anthropic.com>
Parts:
- L3: footprint Inductor_SMD:L_Coilcraft_LPS4018 -> SC:L_Coilcraft_LPS4018
Changed lines of the file:
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@@
   (property "Reference" "L3" (at 71.12 168.91 0) (effects (font (size 1.27 1.27)) (justify left)))
   (property "Value" "10uH LPS4018-103MRC" (at 71.12 171.45 0) (effects (font (size 1.27 1.27)) (justify left)))
-  (property "Footprint" "Inductor_SMD:L_Coilcraft_LPS4018" (at 69.85 170.18 0) (effects (font (size 1.27 1.27)) (hide yes)))
+  (property "Footprint" "SC:L_Coilcraft_LPS4018" (at 69.85 170.18 0) (effects (font (size 1.27 1.27)) (hide yes)))
   (property "MPN" "LPS4018-103MRC" (at 69.85 170.18 0) (effects (font (size 1.27 1.27)) (hide yes)))
   (pin "1")(pin "2")
