File: candidates/claude-oneshot-revA/kicad/10_storage_audio.kicad_sch (KiCad schematic)
At the start: 23 parts, among them J8 DM3AT-SF-PEJM5, U10 TPS22918DBVR, U12 TPS22918DBVR, U23 TPD4E05U06DQAR, U24 TXU0202DCUR

Commit message: candidates: evidence-backed refinement of the Claude one-shot KiCad candidate
Reviewed on origin/main e1f75a3 with KiCad 10.0.6; changes stay inside
candidates/claude-oneshot-revA/ and close no project gate.

- TXU0202 U24: exact TI DCU0008A land (SCES942A pp.32-34) replaces the
  generic KiCad DCU footprint; schematic/symbol footprint fields updated.
- TPS259474L U3 RPW: copper verified against the TI 4225183/A vectors;
  paste now follows the TI stencil example, fab body 2.0 mm.
- ICM-42688-P pin 9 tied to GND (TDK DS-000347 v1.9 Table 10).
- U1/J5 body-courtyard overlap fixed, duplicate vias removed, BMP581
  under-body SCL route removed, SHT40 SDA and 3V3 fragments connected,
  three GND islands stitched, C57 connected, silkscreen refined.
- Removed the unreviewed mask-bridge suppression on U30/U32; findings
  are now visible pending assembler review.
- Before/after ERC, DRC+parity, unconnected and net/pad reconciliation
  reports plus docs/REFINEMENT_2026_09_23.md. Remaining: floating GND at
  U2/U3/U24, SX1262 RF blocker, O05 and the other open gates.

Co-Authored-By: Claude Opus 5.5 <noreply@anthropic.com>
Parts:
- U24: footprint Package_SO:VSSOP-8_2.3x2mm_P0.5mm -> SC:TI_DCU0008A_VSSOP-8_2.3x2mm_P0.5mm_TXU0202
Changed lines of the file:
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@@
   (property "Reference" "U24" (at 33.02 106.68 0) (effects (font (size 1.27 1.27)) (justify left)))
   (property "Value" "TXU0202DCUR" (at 33.02 109.22 0) (effects (font (size 1.27 1.27)) (justify left)))
-  (property "Footprint" "Package_SO:VSSOP-8_2.3x2mm_P0.5mm" (at 43.18 123.19 0) (effects (font (size 1.27 1.27)) (hide yes)))
+  (property "Footprint" "SC:TI_DCU0008A_VSSOP-8_2.3x2mm_P0.5mm_TXU0202" (at 43.18 123.19 0) (effects (font (size 1.27 1.27)) (hide yes)))
   (property "MPN" "TXU0202DCUR" (at 43.18 123.19 0) (effects (font (size 1.27 1.27)) (hide yes)))
   (property "Source" "TI SCES942A (DCU = VSSOP-8 2.3x2.0 mm)" (at 43.18 123.19 0) (effects (font (size 1.27 1.27)) (hide yes)))
