File: candidates/claude-oneshot-revA/kicad/03_rails.kicad_sch (KiCad schematic)
At the start: 24 parts, among them U7 TPS62130ARGTR, U8 TPS7A2030PDBVR, U9 TPS7A2018PDBVR

Commit message: docs: show one-shot candidate renders and schematic in README, fix 3D models
Root README gains a status table for the Claude one-shot candidate, 3D and
enclosure renders, PCB copper view, all 12 schematic sheets as images and
step-by-step instructions (folders) to open the KiCad project or the STEP
files. Candidate README gets the same gallery and KiCad instructions.

3D: envelope STEP models for parts whose footprint had no model in the
KiCad 10.0.6 install (MAX-M10S, ICM-42688-P, MMC5983MA, BMP581, TPD1E0B04,
TPS259474L RPW, TUSB320LAI, Coilcraft inductors, SHT40), so the board STEP
and the Alt+3 view are complete. Routing unchanged; DRC 1 reviewed error,
11 unconnected, parity 0.

Co-Authored-By: Claude Opus 5.5 <noreply@anthropic.com>
Parts:
- L2: footprint Inductor_SMD:L_Coilcraft_XxL4020 -> SC:L_Coilcraft_XxL4020
Changed lines of the file:
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@@
   (property "Reference" "L2" (at 74.93 45.72 0) (effects (font (size 1.27 1.27)) (justify left)))
   (property "Value" "2.2uH XFL4020-222MEB" (at 74.93 48.26 0) (effects (font (size 1.27 1.27)) (justify left)))
-  (property "Footprint" "Inductor_SMD:L_Coilcraft_XxL4020" (at 73.66 46.99 0) (effects (font (size 1.27 1.27)) (hide yes)))
+  (property "Footprint" "SC:L_Coilcraft_XxL4020" (at 73.66 46.99 0) (effects (font (size 1.27 1.27)) (hide yes)))
   (property "MPN" "XFL4020-222MEB" (at 73.66 46.99 0) (effects (font (size 1.27 1.27)) (hide yes)))
   (pin "1")(pin "2")

Commit message: candidates: close floating grounds, swap TPS62130A to RGT0016C, add review notes
Integrates the parallel review work on the Claude one-shot candidate
(candidates/ only; no baseline, locked decision or gate changed):

- GND of U2 (USB ESD), U3 pad 8 (eFuse) and U24 pad 2 connected by local
  re-layout; U7 exposed pad now has 4 vias; GND is one copper group.
- U7 swapped to the TI RGT0016C land (SLVSAG7F p.41) and schematic field
  updated; J1 +0.3 mm move tried and reverted (collides in USB corner).
- Review notes: ESP32/USB-C/buttons audit (all 41 module pads verified),
  TPS62130A footprint, SX1262 E449 native values (topology redraw needed),
  GPIO A5-A8 options (owner decision), assembler mask rules and a dated
  cost snapshot (BRL 200 target infeasible on current parts).
- Final checks: unconnected 2 (SX1262 RF blocker only), parity 0,
  970 pins / 0 mismatches; remaining DRC errors are the U30/U32 mask
  bridges pending the assembler decision.

Co-Authored-By: Claude Opus 5.5 <noreply@anthropic.com>
Parts:
- U7: footprint SC:TI_RGT0016A_VQFN-16_3x3mm_EP1.75x1.75_TPS62130A -> SC:TI_RGT0016C_VQFN-16_3x3mm_EP1.68x1.68_TPS62130A
Changed lines of the file:
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@@
   (property "Reference" "U7" (at 31.75 43.18 0) (effects (font (size 1.27 1.27)) (justify left)))
   (property "Value" "TPS62130ARGTR" (at 31.75 45.72 0) (effects (font (size 1.27 1.27)) (justify left)))
-  (property "Footprint" "SC:TI_RGT0016A_VQFN-16_3x3mm_EP1.75x1.75_TPS62130A" (at 41.91 59.69 0) (effects (font (size 1.27 1.27)) (hide yes)))
+  (property "Footprint" "SC:TI_RGT0016C_VQFN-16_3x3mm_EP1.68x1.68_TPS62130A" (at 41.91 59.69 0) (effects (font (size 1.27 1.27)) (hide yes)))
   (property "MPN" "TPS62130ARGTR" (at 41.91 59.69 0) (effects (font (size 1.27 1.27)) (hide yes)))
   (property "Source" "TI SLVSAG7F" (at 41.91 59.69 0) (effects (font (size 1.27 1.27)) (hide yes)))
