File: candidates/claude-oneshot-revA/kicad/StratosCore_Claude.kicad_pcb (KiCad board)
At the start: 4 copper layers, 60 x 84 mm, 277 parts, among them J1 USB4105-GF-A, J2 BM12B-GHS-TBT (expansion), J3 XF3M-4015-1B (TFT 40p FPC), J4 XF3M-0615-1B (CTP 6p FPC), J5 U.FL-R-SMT-1(60) GNSS, J6 U.FL-R-SMT-1(60) LoRa, J7 U.FL-R-SMT-1(60) ADS-B, J8 DM3AT-SF-PEJM5, Q1 Dual N-MOSFET TBD (O05), Q2 2N7002, SW1 SKSCLCE010 (BUTTON_1 / BOOT), SW2 SKSCLCE010 (BUTTON_2), U1 ESP32-S3-WROOM-1-N16R8, U10 TPS22918DBVR, U11 TPS22918DBVR, U12 TPS22918DBVR, U13 TCA9535PWR, U14 SN74AXC4T245PWR, U15 SN74LVC1G07DBVR, U16 TPS61169DCKR, U17 MAX-M10S-00B, U2 TPD4E05U06DQAR, U20 RP2040, U21 W25Q128JVSIQ, U23 TPD4E05U06DQAR, U24 TXU0202DCUR, U3 TPS259474LRPWR, U30 ICM-42688-P, U31 MMC5983MA, U32 BMP581, U33 SHT40-AD1B-R2, U4 TUSB320LAIRWBR, U40 SX1262IMLTRT, U41 PE4259, U5 S-8252 (product code TBD, O05), U50 BLB01, U52 BLB01, U54 ADL5513ACPZ-R7, U55 MCP6566T-E/OT, U6 BQ25887RGER, U7 TPS62130ARGTR, U8 TPS7A2030PDBVR, U9 TPS7A2018PDBVR, Y1 12MHz ABM8-272-T3, Y2 32 MHz (CL 10pF) MPN TBD

Commit message: candidate: stitch floating GND pads U2/U3/U24 to In1 plane
- U24.2 (TXU0202): 0.2mm track staircase + 0.45/0.2 via into In1 plane
- U2.3 (TPD4E05U06): direct 0.127mm track + 0.35/0.2 via (0.330mm d_min)
- U3.8 (TPS259474L): 0.127mm staircase via 0.35/0.2 landing on In1
- In2.In1 landing verified by PointInside on anchored GND fill outline
- via clearances: 0.15 full-class / 0.127 JLC-class with geometric proof

DRC after (KiCad 10.0.6): unconnected 5 -> 2 (only intended LORA_RFO/RFI_P
TBD stubs), 0 new clearance/short/hole-to-hole items, schematic parity 0.
Remaining violations pre-exist: 199 solder_mask_bridge (assembler gate),
117 silk (cosmetic), 1 track_dangling (LoRa TBD).
Routing:
- net GND: track 657.0 -> 665.0 mm, vias 291 -> 294

Commit message: candidate: merge artifact removed — clean GND stitch board + U7 RGT0016C
Replaces the text-merge artifact (4 shorts / 10 clearances from mixing two
copper generations) with the verified board: v19 GND stitches (U2 via
0.35/0.2, U24 via 0.45/0.2, U3 staircase+via) + U7 footprint block swapped
to RGT0016C (SLVSAG7F p.41) via s-expression surgery, no copper merge.

DRC (KiCad 10.0.6): unconnected 2 (LORA_RFO/RFI_P TBD only), 0 shorts,
0 hole violations, parity 0. Residual: 10 clearance items at U3 east
rail-stair chords + TP1 island (cause analyzed; fix queued: orthogonal
re-route with 0.55mm TP1 keepout, goal via 0.4/0.2).
Routing:
- net GND: track 665.0 -> 663.6 mm, vias 294 -> 288
- net BUCK_SW: track 14.5 -> 13.6 mm
- net SD_CT: track 13.4 -> 12.7 mm
